File: hardware/VitalX-ESP/VitalX-ESP.kicad_sch (KiCad schematic)
At the start: 55 parts, among them J1 ECG Probe, J2 GSR Probe, J3 UART, J4 JTAG, Q1 BSS138, SW2 Reset, U1 AD8232ACPZ-R7, U3 ADP160AUJZ-1.8-R7, U4 ADPD144RI-ACEZ-RL, U5 AMS1117-3.3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

Commit message: [nightly] Finalize schematic.
Added power connector.
Parts:
- added J5: Power terminal, TerminalBlock:TerminalBlock_bornier-2_P5.08mm, symbol Connector:Screw_Terminal_01x02
- J1: footprint AUDIO_SJ2-3574A-SMT-TR:SJ2-3574A-SMT-TR -> Connector_Audio:Jack_3.5mm_PJ320D_Horizontal
Connections:
- net +5V: now also J5.1 (Pin_1)
- net GND: now also J5.2 (Pin_2)
Other:
- moved on the sheet: C12, C7, C8, U3, U5
