File: hardware/VitalX-ESP/VitalX-ESP.kicad_pcb (KiCad board)
At the start: 2 copper layers, 25 parts, among them J1 ECG Probe, U1 AD8232ACPZ-R7, U2 ESP32-WROOM-32U, U3 ADP160AUJZ-1.8-R7

Commit message: [nightly] Initial PCB layout.
4 layer stack up:
- Signal
- GND
- GND
- Signal
Currently working on ECG Block.
Parts:
- removed U2: ESP32-WROOM-32U, RF_Module:ESP32-WROOM-32U
- added C10: 1u, Capacitor_SMD:C_0603_1608Metric, F.Cu at (157.0, 76.5)
- added C11: 10u, Capacitor_SMD:C_0603_1608Metric, F.Cu at (165.0, 76.3)
- added C12: 1u, Capacitor_SMD:C_0603_1608Metric, F.Cu at (167.0, 127.8)
- added C13: 100n, Capacitor_SMD:C_0603_1608Metric, F.Cu at (105.3, 134.0)
- added C14: 22u, Capacitor_SMD:C_0603_1608Metric, F.Cu at (120.0, 56.3)
- added C15: 100n, Capacitor_SMD:C_0603_1608Metric, F.Cu at (115.0, 55.8)
- added C16: 1u, Capacitor_SMD:C_0603_1608Metric, F.Cu at (148.0, 56.2)
- added C17: 100n, Capacitor_SMD:C_0603_1608Metric, F.Cu at (112.0, 85.2)
- added C7: 1u, Capacitor_SMD:C_0603_1608Metric, F.Cu at (184.0, 129.2)
- added C8: 1u, Capacitor_SMD:C_0603_1608Metric, F.Cu at (193.0, 129.2)
- added C9: 1.5n, Capacitor_SMD:C_0603_1608Metric, F.Cu at (79.8, 87.8)
- added J2: GSR Probe, Connector_PinHeader_2.54mm:PinHeader_1x02_P2.54mm_Vertical_SMD_Pin1Left, F.Cu at (117.3, 130.7)
- added J3: UART, Connector_PinHeader_2.54mm:PinHeader_1x04_P2.54mm_Vertical_SMD_Pin1Left, F.Cu at (190.7, 54.8)
- added J4: JTAG, Connector_PinHeader_2.54mm:PinHeader_1x04_P2.54mm_Vertical_SMD_Pin1Left, F.Cu at (190.7, 72.7)
- added J5: Power terminal, TerminalBlock:TerminalBlock_bornier-2_P5.08mm, F.Cu at (171.5, 141.0)
- added JP1: Boot Mode, Connector_PinHeader_2.54mm:PinHeader_1x02_P2.54mm_Vertical_SMD_Pin1Left, F.Cu at (104.7, 63.3)
- added Q1: BSS138, Package_TO_SOT_SMD:SOT-23, F.Cu at (161.5, 82.8)
- added R16: 10K, Resistor_SMD:R_0603_1608Metric, F.Cu at (166.0, 82.7)
- added R17: 10K, Resistor_SMD:R_0603_1608Metric, F.Cu at (157.0, 82.9)
- added R18: 10K, Resistor_SMD:R_0603_1608Metric, F.Cu at (146.0, 72.2)
- added R19: 10K, Resistor_SMD:R_0603_1608Metric, F.Cu at (150.0, 73.8)
- added R20: 100k, Resistor_SMD:R_0603_1608Metric, F.Cu at (110.3, 127.9)
- added R21: 100k, Resistor_SMD:R_0603_1608Metric, F.Cu at (110.3, 132.7)
- added R22: 100k, Resistor_SMD:R_0603_1608Metric, F.Cu at (93.3, 133.0)
- added R23: 100k, Resistor_SMD:R_0603_1608Metric, F.Cu at (99.3, 128.0)
- added R24: 10K, Resistor_SMD:R_0603_1608Metric, F.Cu at (153.0, 56.2)
- added R25: 10K, Resistor_SMD:R_0603_1608Metric, F.Cu at (133.0, 83.0)
- added SW2: Reset, Button_Switch_THT:SW_PUSH_1P1T_6x3.5mm_H5.0_APEM_MJTP1250, F.Cu at (105.0, 82.8)
- added U4: ADPD144RI-ACEZ-RL, ADPD144RI:CE-12-2_ADI, F.Cu at (161.0, 73.8)
- added U5: AMS1117-3.3, Package_TO_SOT_SMD:SOT-223-3_TabPin2, F.Cu at (173.8, 129.0)
- added U6: MCP601-xOT, Package_TO_SOT_SMD:SOT-23-5, F.Cu at (99.3, 134.0)
- added U7: ESP32-S2-WROOM, ESP32-S2-WROOM:esp32-s2-wrooom, F.Cu at (133.7, 63.3)
- J1: footprint Connector_Audio:Jack_3.5mm_CUI_SJ2-3593D-SMT_Horizontal -> AUDIO_SJ2-3593D-SMT-TR:SJ2-3593D-SMT-TR
- R13, R14: value 1M -> 10M
- moved U3 190.6 mm to (188.4, 129.4)
- moved R15 128.7 mm to (142.0, 83.0), turned to -90 degrees
- moved J1 92.1 mm to (48.0, 90.8), turned to -90 degrees
- moved C3 91.5 mm to (74.3, 95.6), turned to -90 degrees
- moved R11 88.1 mm to (77.1, 95.6), turned to 90 degrees
- moved C4 87.7 mm to (71.5, 95.6), turned to -90 degrees
- moved C1 87.4 mm to (67.5, 90.9), turned to 180 degrees
- moved R12 85.2 mm to (79.8, 91.9), turned to -90 degrees
- moved R9 84.9 mm to (79.0, 84.8), turned to 180 degrees
- moved R8 84.0 mm to (75.1, 98.4), turned to 180 degrees
- moved C5 83.2 mm to (76.1, 87.2), turned to 90 degrees
- moved R10 81.5 mm to (79.0, 82.6)
- moved C2 81.2 mm to (68.3, 84.6), turned to 90 degrees
- moved R2 80.9 mm to (63.6, 88.7)
- moved R5 80.6 mm to (67.4, 93.0)
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Connections:
- R10 pad 2: ECG_OUT -> Net-(C9-Pad2)
- R9 pad 1: ECG_OUT -> Net-(C9-Pad2)
- U3 pad 1: unconnected-(U3-VIN-Pad1) -> +3V3
- U3 pad 2: unconnected-(U3-GND-Pad2) -> GND
- U3 pad 3: unconnected-(U3-EN-Pad3) -> +3V3
- U3 pad 5: unconnected-(U3-VOUT-Pad5) -> +1V8
Routing:
- net Net-(R6-Pad2): track 0.00 -> 35.2 mm, vias 0 -> 2
- net Net-(U1-OPAMP+): track 0.00 -> 26.1 mm, vias 0 -> 2
- net /REFIN: track 0.00 -> 15.0 mm, vias 0 -> 2
- net /SW: track 0.00 -> 14.9 mm
- net Net-(U1-OPAMP-): track 0.00 -> 14.4 mm
- net /IAOUT: track 0.00 -> 12.2 mm
- net /REFOUT: track 0.00 -> 11.4 mm
- net ECG_OUT: track 0.00 -> 10.2 mm
- net Net-(U1-HPSENSE): track 0.00 -> 6.73 mm
- net RA: track 0.00 -> 6.62 mm
- net /IN-: track 0.00 -> 5.93 mm
- net /IN+: track 0.00 -> 5.85 mm
- net Net-(U1-RLD): track 0.00 -> 5.67 mm
- net Net-(U1-RLDFB): track 0.00 -> 5.12 mm
- net Net-(C9-Pad2): track 0.00 -> 4.43 mm
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Other:
- copper layers 2 -> 4

Commit message: [nightly] Inital signals routing.
First iteration of signals (only) routing.
Parts:
- J1: value ECG Probe -> EGC Probe; footprint AUDIO_SJ2-3593D-SMT-TR:SJ2-3593D-SMT-TR -> Connector_Audio:Jack_3.5mm_KoreanHropartsElec_PJ-320D-4A_Horizontal
- moved R4 83.2 mm to (138.0, 104.8)
- moved R2 73.3 mm to (135.1, 104.8), turned to 90 degrees
- moved R3 73.0 mm to (130.4, 104.8)
- moved R5 72.5 mm to (139.5, 101.0), turned to 90 degrees
- moved R1 72.0 mm to (133.3, 104.8), turned to 90 degrees
- moved C1 70.6 mm to (137.4, 100.9), turned to -90 degrees
- moved C4 70.6 mm to (142.1, 96.9), turned to 0 degrees
- moved R8 70.0 mm to (144.9, 93.3), turned to -90 degrees
- moved R21 68.6 mm to (113.0, 64.2), turned to 0 degrees
- moved C3 67.8 mm to (142.1, 94.1), turned to 0 degrees
- moved C13 67.5 mm to (114.6, 67.1), turned to 180 degrees
- moved R11 65.2 mm to (142.1, 91.3), turned to 180 degrees
- moved U6 64.8 mm to (115.4, 71.2), turned to -90 degrees
- moved C2 64.7 mm to (131.1, 100.1), turned to 180 degrees
- moved J1 64.7 mm to (111.5, 103.0), turned to 90 degrees
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Connections:
- R1 pad 1: LA -> /IN+
- R1 pad 2: /IN+ -> LA
- U7 pad 10: unconnected-(U7-IO7-Pad10) -> /GSR_OUT
- U7 pad 14: /GSR_OUT -> ECG_OUT
- U7 pad 23: unconnected-(U7-IO20-Pad23) -> /LOD+
- U7 pad 24: unconnected-(U7-IO21-Pad24) -> /LOD-
- U7 pad 39: /LOD- -> unconnected-(U7-IO45-Pad39)
- U7 pad 4: ECG_OUT -> unconnected-(U7-IO1-Pad4)
- U7 pad 40: /LOD+ -> unconnected-(U7-IO46-Pad40)
Routing:
- net RL: track 0.00 -> 50.1 mm
- net /TCK: track 0.00 -> 32.9 mm
- net /TDI: track 0.00 -> 31.5 mm
- net Net-(J3-Pin_2): track 0.00 -> 29.2 mm
- net /TDO: track 0.00 -> 28.6 mm
- net /TMS: track 0.00 -> 27.8 mm
- net ECG_OUT: track 10.2 -> 36.6 mm, vias 0 -> 2
- net Net-(J3-Pin_3): track 0.00 -> 25.5 mm
- net RA: track 6.62 -> 31.5 mm
- net LA: track 2.98 -> 26.0 mm
- net /SDN: track 0.00 -> 22.6 mm, vias 0 -> 2
- net +3V3: track 0.00 -> 19.3 mm
- net /PPG_INT: track 0.00 -> 17.2 mm
- net /SCL: track 0.00 -> 16.9 mm
- net /LOD-: track 0.00 -> 16.6 mm, vias 0 -> 2
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Other:
- board outline added: 73 x 63 mm
- board text added: "Considering USB connector."

Commit message: [nightly] Finalize board layout.
Parts:
- moved J5 11.4 mm to (156.9, 102.6), turned to 0 degrees
- moved C5 0.38 mm to (132.6, 92.5), turned to 180 degrees
Connections:
- C5 pad 2: +3.3V -> +3V3
- R13 pad 2: +3.3V -> +3V3
- R15 pad 2: +3.3V -> +3V3
- R3 pad 2: +3.3V -> +3V3
- R4 pad 2: +3.3V -> +3V3
- U1 pad 15: +3.3V -> +3V3
- U1 pad 17: +3.3V -> +3V3
- U7 pad : (no net) -> GND
Routing:
- net +3V3: track 19.3 -> 317.3 mm, vias 0 -> 14
- net GND: track 13.9 -> 83.7 mm, vias 0 -> 22
- net +1V8: track 2.33 -> 39.2 mm, vias 0 -> 3
- net +5V: track 15.0 -> 7.56 mm
- added copper zone on In1.Cu, net GND
- added copper zone on In2.Cu, net GND
Other:
- outline, holes or cut-outs redrawn

Commit message: [nightly] Change ECG Probe footprint.
Changes in accordance with reference design.
- https://www.snapeda.com/parts/SJ2-3593D-SMT-TR/CUI%20Devices/view-part/?ref=mouser
- https://easyeda.com/editor#project_id=8294b8a1d6874413ae900972098163d6
Parts:
- J1: value EGC Probe -> ECG Probe; footprint Connector_Audio:Jack_3.5mm_KoreanHropartsElec_PJ-320D-4A_Horizontal -> AUDIO_SJ2-3593D-SMT-TR:SJ2-3593D-SMT-TR
- moved J1 7.93 mm to (109.9, 95.2), turned to 0 degrees
Connections:
- J1 pad S: GND -> RL
- J1 pad T: RL -> RA
Routing:
- net GND: track 83.7 -> 74.7 mm
- net LA: track 26.0 -> 32.0 mm
- net RL: track 50.1 -> 45.8 mm
- net RA: track 31.5 -> 28.4 mm
